Commit message: modified & updated & fixed bugs

File: test/urdf/car-robot-chassis.xacro (robot description, xacro)
@@ -21,7 +21,6 @@
 		</collision>
 		<inertial>
-			<mass value="0.4" />
-			<inertia ixx="0.00048333" iyy="0.0013367" izz="0.0018133"
-			ixy="0" ixz="0" iyz="0"/>
+			<mass value="0.8" />
+			<inertia ixx="0.00048333" iyy="0.0013367" izz="0.0018133" ixy="0" ixz="0" iyz="0"/>
 		</inertial>
 	</link>

File: test/urdf/car-robot-gazebo.xacro (robot description, xacro)
@@ -6,6 +6,6 @@
   <xacro:macro name="color_wheel" params="x_position y_position">
     <gazebo reference="${x_position}-${y_position}-wheel-link">
-      <mu1>10000.0</mu1>
-      <mu2>10000.0</mu2>
+      <mu1>5000.0</mu1>
+      <mu2>5000.0</mu2>
       <material>Gazebo/Purple</material>
     </gazebo>
@@ -13,19 +13,32 @@
   <!-- Differential drive plugin -->
   <gazebo>
-    <plugin name="differential_drive_controller" filename="libgazebo_ros_diff_drive.so">
-      <alwaysOn>true</alwaysOn>
-      <updateRate>100</updateRate>
+    <plugin name="skid_steer_drive" filename="libgazebo_ros_diff_drive.so">
+      <!-- Wheel joints -->
+      <num_wheel_pairs>2</num_wheel_pairs>
+      <left_joint>joint-chassis-front-left-wheel</left_joint>
       <left_joint>joint-chassis-rare-left-wheel</left_joint>
+      <right_joint>joint-chassis-front-right-wheel</right_joint>
       <right_joint>joint-chassis-rare-right-wheel</right_joint>
+      <!-- Kinematics -->
       <wheel_separation>${chassis_width}</wheel_separation>
       <wheel_diameter>${2 * wheel_radius}</wheel_diameter>
-      <torque>0.1</torque>
-      <commandTopic>cmd_vel</commandTopic>
-      <odometryTopic>odom</odometryTopic>
-      <odometryFrame>odom</odometryFrame>
-      <robotBaseFrame>base_link</robotBaseFrame>
-      <publishWheelTF>true</publishWheelTF>
-      <publishOdom>true</publishOdom>
-      <publishWheelJointState>true</publishWheelJointState>
+      <!-- Limits -->
+      <max_wheel_torque>4.0</max_wheel_torque>      <!-- Adjust as per your model -->
+      <max_wheel_acceleration>0.2</max_wheel_acceleration>      <!-- Optional -->
+      <!-- Odometry & Frames -->
+      <odometry_topic>odom</odometry_topic>      <!-- Important -->
+      <odometry_frame>odom</odometry_frame>      <!-- Important -->
+      <robot_base_frame>base_link</robot_base_frame>      <!-- Important -->
+      <publish_odom>true</publish_odom>      <!-- Crucial -->
+      <publish_odom_tf>true</publish_odom_tf>      <!-- Crucial -->
+      <!-- <ros>
+        <namespace>/</namespace>
+        <argument>/cmd_vel:=cmd_vel</argument>
+        <argument>/odom:=odom</argument>
+      </ros> -->
+      <command_topic>cmd_vel</command_topic>
+      <!-- Misc -->
+      <publish_wheel_joint_state>true</publish_wheel_joint_state>
+      <update_rate>20.0</update_rate>      <!-- Stable frequency -->
     </plugin>
   </gazebo>
@@ -72,6 +85,6 @@
             <samples>360</samples>
             <resolution>1</resolution>
-            <min_angle>-1.5707</min_angle> <!-- -90 degrees (left) -->
-			<max_angle>1.5707</max_angle>  <!-- +90 degrees (right) -->
+            <min_angle>-1.5707</min_angle>            <!-- -90 degrees (left) -->
+            <max_angle>1.5707</max_angle>            <!-- +90 degrees (right) -->
           </horizontal>
         </scan>
@@ -87,9 +100,9 @@
         </noise>
       </ray>
-       <plugin name="gazebo_ros_head_hokuyo_controlle" filename="libgazebo_ros_ray_sensor.so" >
-          <ros>
+      <plugin name="gazebo_ros_head_hokuyo_controlle" filename="libgazebo_ros_ray_sensor.so">
+        <ros>
           <remapping>~/out:=/scan</remapping>
-          </ros>
-          <output_type>sensor_msgs/LaserScan</output_type>
+        </ros>
+        <output_type>sensor_msgs/LaserScan</output_type>
       </plugin>
     </sensor>

File: test/urdf/car-robot-inertia.xacro (robot description, xacro)
@@ -1,11 +1,11 @@
 <?xml version='1.0'?>
-<robot xmlns:xacro ="http://www.ros.org/wiki/xacro" name="car_robot_inertia">
+<robot xmlns:xacro="http://www.ros.org/wiki/xacro" name="car_robot_inertia">
+	<!-- Box Inertia -->
 	<xacro:macro name="box_inertia" params="mass L W H">
-		<inertia ixx="${1/12 * mass * (L**2 + W**2 )}" iyy="${1/12 * mass * (H**2 + W**2 )}" izz="${1/12 * mass * (L**2 + H**2 )}"
-		ixy="0" ixz="0" iyz="0"/>
+		<inertia ixx="${(1.0/12.0) * mass * (L*L + W*W)}" iyy="${(1.0/12.0) * mass * (H*H + W*W)}" izz="${(1.0/12.0) * mass * (L*L + H*H)}" ixy="0" ixz="0" iyz="0"/>
 	</xacro:macro>
+	<!-- Cylinder Inertia -->
 	<xacro:macro name="cylinder_inertia" params="mass R H">
-		<inertia ixx="${1/12 * mass * (3 * R**2 + H**2 )}" iyy="${1/12 * mass * (3 * R**2 + H**2 )}" izz="${0.5 * (mass * R**2 )}"
-		ixy="0" ixz="0" iyz="0"/>
+		<inertia ixx="${(1.0/12.0) * mass * (3*R*R + H*H) + (1.0/4.0) * mass * R*R}" iyy="${(1.0/12.0) * mass * (3*R*R + H*H) + (1.0/4.0) * mass * R*R}" izz="${(1.0/2.0) * mass * R*R}" ixy="0" ixz="0" iyz="0"/>
 	</xacro:macro>
 </robot>

File: test/urdf/car-robot-params.xacro (robot description, xacro)
@@ -1,8 +1,8 @@
 <?xml version='1.0'?>
-<robot xmlns:xacro ="http://www.ros.org/wiki/xacro" >
+<robot xmlns:xacro ="http://www.ros.org/wiki/xacro">
 	<xacro:property name="chassis_length" value="0.14" />
 	<xacro:property name="chassis_width" value="0.12" />
 	<xacro:property name="chassis_height" value="0.01" />
-	<xacro:property name="chassis_mass" value="0.4" />
+	<xacro:property name="chassis_mass" value="0.8" />
 	<xacro:property name="wheel_radius" value="0.02" />
 	<xacro:property name="wheel_height" value="0.01" />

File: test/urdf/car-robot-wheel.xacro (robot description, xacro)
@@ -5,10 +5,10 @@
 	</material>
 	<xacro:macro name="wheel" params="x_position y_position x_reflect y_reflect">
-	<!-- ${x_position}-${y_position}-wheel-link -->
+		<!-- ${x_position}-${y_position}-wheel-link -->
 		<link name="${x_position}-${y_position}-wheel-link">
 			<visual>
 				<origin xyz="0 0 0" rpy="${pi * 0.5} 0 0" />
 				<geometry>
-					<cylinder radius ="${wheel_radius}"  length="${wheel_height}" />
+					<cylinder radius ="${wheel_radius}" length="${wheel_height}" />
 				</geometry>
 				<material name="blue" />
@@ -17,11 +17,10 @@
 				<origin xyz="0 0 0" rpy="${pi * 0.5} 0 0" />
 				<geometry>
-					<cylinder radius ="${wheel_radius}"  length="${wheel_height}" />
+					<cylinder radius ="${wheel_radius}" length="${wheel_height}" />
 				</geometry>
 			</collision>
 			<inertial>
-				<origin xyz="0 0 0" rpy="${pi * 0.5} 0 0" />
 				<mass value="${wheel_mass}" />
-				<xacro:cylinder_inertia  mass="${wheel_mass}" R="${wheel_radius}" H="${wheel_height}" />
+				<inertia ixx="0.0001" ixy="0.0" ixz="0.0" iyy="0.0002" iyz="0.0" izz="0.0003"/>
 			</inertial>
 		</link>

File: test/urdf/car-robot.xacro (robot description, xacro)
@@ -1,4 +1,4 @@
 <?xml version='1.0'?>
-<robot xmlns:xacro ="http://www.ros.org/wiki/xacro" name="car-robot" >
+<robot xmlns:xacro ="http://www.ros.org/wiki/xacro" name="car-robot">
 	<xacro:include filename="$(find test)/urdf/car-robot-params.xacro" />
 	<xacro:include filename="$(find test)/urdf/car-robot-inertia.xacro" />
